Commit message: feat: replace LeKiwi arm model with SO-101

File: URDF/LeKiwi.urdf (robot description, URDF)
Before this commit: robot LeKiwi, 45 links, 44 joints
Links:
- removed link Base_08q-v1
- removed link Camera-Model-v3-1
- removed link Moving_Jaw_08d-v1
- removed link Passive_Horn_01-v1
- removed link Rotation_Pitch_08i-v1
- removed link SO_ARM100_08k_116_Square-v1
- removed link SO_ARM100_08k_Asym_Mirror_Clip-v1
- removed link SO_ARM100_08k_Mirror-v1
- removed link STS3215_03a-v1
- removed link STS3215_03a-v1-1
- removed link STS3215_03a-v1-2
- removed link STS3215_03a-v1-3
- removed link STS3215_03a-v1-4
- removed link STS3215_03a_Wrist_Roll-v1
- removed link WaveShare_Mounting_Plate_01d-v1
- removed link Wrist-Camera-Mount-v11
- removed link Wrist_Roll_08c-v1
- removed link Wrist_Roll_Pitch_08i-v1
- added link so101_base_link, mass 0.147; collision mesh filename=meshes/so101/base_motor_holder_so101_v1.stl; collision mesh filename=meshes/so101/base_so101_v2.stl
- added link so101_gripper_frame_link, mass 1e-9
- added link so101_gripper_link, mass 0.087; collision mesh filename=meshes/so101/sts3215_03a_v1.stl; collision mesh filename=meshes/so101/wrist_roll_follower_so101_v1.stl
- added link so101_lower_arm_link, mass 0.104; collision mesh filename=meshes/so101/motor_holder_so101_wrist_v1.stl; collision mesh filename=meshes/so101/sts3215_03a_v1.stl
- added link so101_moving_jaw_link, mass 0.012; collision mesh filename=meshes/so101/moving_jaw_so101_v1.stl; visual mesh filename=meshes/so101/moving_jaw_so101_v1.stl
- added link so101_shoulder_link, mass 0.100006; collision mesh filename=meshes/so101/motor_holder_so101_base_v1.stl; collision mesh filename=meshes/so101/rotation_pitch_so101_v1.stl
- added link so101_upper_arm_link, mass 0.103; collision mesh filename=meshes/so101/sts3215_03a_v1.stl; collision mesh filename=meshes/so101/upper_arm_so101_v1.stl
- added link so101_wrist_link, mass 0.079; collision mesh filename=meshes/so101/sts3215_03a_no_horn_v1.stl; collision mesh filename=meshes/so101/wrist_roll_pitch_so101_v2.stl
Joints:
- removed joint Base_08q-v1_Rigid-43
- removed joint Base_08q-v1_Rigid-44
- removed joint Base_08q-v1_Rigid-47
- removed joint Rotation_Pitch_08i-v1_Rigid-46
- removed joint Rotation_Pitch_08i-v1_Rigid-48
- removed joint SO_ARM100_08k_116_Square-v1_Rigid-50
- removed joint SO_ARM100_08k_Mirror-v1_Rigid-52
- removed joint Wrist-Camera-Mount-v11_Rigid-71
- removed joint Wrist_Roll_08c-v1_Rigid-56
- removed joint Wrist_Roll_08c-v1_Rigid-58
- removed joint Wrist_Roll_Pitch_08i-v1_Rigid-54
- removed joint base_plate_layer2-v3_Rigid-42
- added joint so101_gripper_frame_joint: type fixed, parent so101_gripper_link, child so101_gripper_frame_link, origin xyz=-0.0079 -0.000218121 -0.0981274 rpy=0 3.14159 0, axis 0 0 0
- added joint so101_mount: type fixed, parent base_plate_layer2-v3, child so101_base_link, origin xyz=0.0388353 0.06714801 0.007 rpy=0 0 3.14159
- joint arm_elbow_flex: axis 1.0 0.0 0.0 -> 0 0 1; child SO_ARM100_08k_Mirror-v1 -> so101_lower_arm_link; limit (none) -> lower=-1.69 upper=1.69 effort=10 velocity=10; origin xyz=0.0346 -0.013069710000000002 0.03178184000000002 rpy=-6.842277657836021e-49 -3.4512664603419266e-31 -1.3877787807814457e-17 -> xyz=-0.11257 -0.028 1.73763e-16 rpy=-3.63608e-16 8.74301e-16 1.5708; parent STS3215_03a-v1-2 -> so101_upper_arm_link; type continuous -> revolute
- joint arm_gripper: axis -2.74128770133849e-31 -0.9063079999999999 -0.422618 -> 0 0 1; child Moving_Jaw_08d-v1 -> so101_moving_jaw_link; limit (none) -> lower=-0.174533 upper=1.74533 effort=10 velocity=10; origin xyz=-0.032799999999999996 -0.023912249999999986 0.027026410000000018 rpy=-1.5707963267948968 3.944304526105059e-31 -1.9721522630525295e-31 -> xyz=0.0202 0.0188 -0.0234 rpy=1.5708 -5.24284e-08 -1.41553e-15; parent STS3215_03a-v1-4 -> so101_gripper_link; type continuous -> revolute
- joint arm_shoulder_lift: axis 1.0 0.0 0.0 -> 0 0 1; child SO_ARM100_08k_116_Square-v1 -> so101_upper_arm_link; limit (none) -> lower=-1.74533 upper=1.74533 effort=10 velocity=10; origin xyz=0.0346 0.010249999999999987 -0.032799999999999975 rpy=3.141592653589793 1.7181275903033976e-32 -3.1373434374976504e-48 -> xyz=-0.0303992 -0.0182778 -0.0542 rpy=-1.5708 -1.5708 0; parent STS3215_03a-v1-1 -> so101_shoulder_link; type continuous -> revolute
- joint arm_shoulder_pan: axis -3.944304526105059e-31 3.944304526105059e-31 1.0 -> 0 0 1; child Rotation_Pitch_08i-v1 -> so101_shoulder_link; limit (none) -> lower=-1.91986 upper=1.91986 effort=10 velocity=10; origin xyz=-0.010250000000000084 0.03459999999999999 -0.032799999999999996 rpy=1.5707963267948966 -2.781046729970605e-32 3.94430452610506e-31 -> xyz=0.0388353 -8.97657e-09 0.0624 rpy=3.14159 4.18253e-17 -3.14159; parent STS3215_03a-v1 -> so101_base_link; type continuous -> revolute
- joint arm_wrist_flex: axis 1.0 0.0 9.860761315262648e-32 -> 0 0 1; child Wrist_Roll_Pitch_08i-v1 -> so101_wrist_link; limit (none) -> lower=-1.65806 upper=1.65806 effort=10 velocity=10; origin xyz=0.0346 -0.03408158 0.004398620000000015 rpy=3.1415926535897922 9.860761315262648e-32 -9.503163413661107e-47 -> xyz=-0.1349 0.0052 3.62355e-17 rpy=4.02456e-15 8.67362e-16 -1.5708; parent STS3215_03a-v1-3 -> so101_lower_arm_link; type continuous -> revolute
- joint arm_wrist_roll: axis 0.0 0.42261799999999994 -0.9063079999999999 -> 0 0 1; child Wrist_Roll_08c-v1 -> so101_gripper_link; limit (none) -> lower=-2.74385 upper=2.84121 effort=10 velocity=10; origin xyz=-0.028999999999999998 0.00810632 0.006869499999999995 rpy=3.141592653589793 -0.0 0.0 -> xyz=5.55112e-17 -0.0611 0.0181 rpy=1.5708 0.0486795 3.14159; parent STS3215_03a_Wrist_Roll-v1 -> so101_wrist_link; type continuous -> revolute
