Commit message: fix(urdf): generate LeKiwi.urdf and fail on a stale committed model
URDF/LeKiwi.urdf was the untouched upstream model (old Pi case, no sensors,
old arm pose and masses) while consumers read it as the robot. Keep it as
URDF/LeKiwi.baseline.urdf for the migration and semantics checks, and have
export_robot.sh write the plain-URDF expansion of the Xacro instead.

verify_robot.sh now checks the manifest and compares its rebuild with the
committed Xacro, URDF and meshes (meshes as canonical triangle sets, since
exports reorder triangles). That removed three committed meshes no export
produces: the removed Pi case and the superseded SO-101 wrist.

Co-Authored-By: Claude Opus 5.5 (1M context) <noreply@anthropic.com>

File: URDF/LeKiwi.urdf (robot description, URDF)
Before this commit: robot LeKiwi, 35 links, 34 joints
Links:
- removed link Bottom-V2-v3
- removed link Top-V2-v2
- added link astra_pro_compact_mount; collision mesh filename=meshes/reauthored/astra_pro_compact_mount.stl scale=0.001 0.001 0.001; visual mesh filename=meshes/reauthored/astra_pro_compact_mount.stl scale=0.001 0.001 0.001
- added link ld06_body; collision mesh filename=meshes/reauthored/ld06_body.stl scale=0.001 0.001 0.001; visual mesh filename=meshes/reauthored/ld06_body.stl scale=0.001 0.001 0.001
- added link robotskin_lidar_mount; collision mesh filename=meshes/reauthored/robotskin_lidar_mount.stl scale=0.001 0.001 0.001; visual mesh filename=meshes/reauthored/robotskin_lidar_mount.stl scale=0.001 0.001 0.001
- added link rpi5_table; collision mesh filename=meshes/reauthored/rpi5_table.stl scale=0.001 0.001 0.001; visual mesh filename=meshes/reauthored/rpi5_table.stl scale=0.001 0.001 0.001
- added link rpi5_through_plate; collision mesh filename=meshes/reauthored/rpi5_through_plate.stl scale=0.001 0.001 0.001; visual mesh filename=meshes/reauthored/rpi5_through_plate.stl scale=0.001 0.001 0.001
- added link rpi5_usb_carrier; collision mesh filename=meshes/reauthored/rpi5_usb_carrier.stl scale=0.001 0.001 0.001; visual mesh filename=meshes/reauthored/rpi5_usb_carrier.stl scale=0.001 0.001 0.001
- link 4-Omni-Directional-Wheel_Single_Body-v1: geometry collision mesh filename=meshes/reauthored/4-Omni-Directional-Wheel_Single_Body-v1.s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 scale=0.001 0.001 0.001; visual mesh filename=meshes/reauthored/4-Omni-Directional-Wheel_Single_Body-v1.s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 scale=0.001 0.001 0.001
- link 4-Omni-Directional-Wheel_Single_Body-v1-1: geometry collision mesh filename=meshes/reauthored/4-Omni-Directional-Wheel_Single_Body-v1-1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 scale=0.001 0.001 0.001; visual mesh filename=meshes/reauthored/4-Omni-Directional-Wheel_Single_Body-v1-1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 scale=0.001 0.001 0.001
- link 4-Omni-Directional-Wheel_Single_Body-v1-2: geometry collision mesh filename=meshes/reauthored/4-Omni-Directional-Wheel_Single_Body-v1-2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 scale=0.001 0.001 0.001; visual mesh filename=meshes/reauthored/4-Omni-Directional-Wheel_Single_Body-v1-2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 scale=0.001 0.001 0.001
- link 94868A713_NO-THREADS_Female-Threaded-Hex-Standoff: geometry collision mesh filename=meshes/reauthored/94868A713_NO-THREADS_Female-Threaded-Hex-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 scale=0.001 0.001 0.001; visual mesh filename=meshes/reauthored/94868A713_NO-THREADS_Female-Threaded-Hex-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 scale=0.001 0.001 0.001
- link 94868A713_NO-THREADS_Female-Threaded-Hex-Standoff-1: geometry collision mesh filename=meshes/reauthored/94868A713_NO-THREADS_Female-Threaded-Hex-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 scale=0.001 0.001 0.001; visual mesh filename=meshes/reauthored/94868A713_NO-THREADS_Female-Threaded-Hex-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 scale=0.001 0.001 0.001
- link 94868A713_NO-THREADS_Female-Threaded-Hex-Standoff-2: geometry collision mesh filename=meshes/reauthored/94868A713_NO-THREADS_Female-Threaded-Hex-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 scale=0.001 0.001 0.001; visual mesh filename=meshes/reauthored/94868A713_NO-THREADS_Female-Threaded-Hex-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 scale=0.001 0.001 0.001
- link 94868A713_NO-THREADS_Female-Threaded-Hex-Standoff-3: geometry collision mesh filename=meshes/reauthored/94868A713_NO-THREADS_Female-Threaded-Hex-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 scale=0.001 0.001 0.001; visual mesh filename=meshes/reauthored/94868A713_NO-THREADS_Female-Threaded-Hex-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 scale=0.001 0.001 0.001
- link 94868A713_NO-THREADS_Female-Threaded-Hex-Standoff-4: geometry collision mesh filename=meshes/reauthored/94868A713_NO-THREADS_Female-Threaded-Hex-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 scale=0.001 0.001 0.001; visual mesh filename=meshes/reauthored/94868A713_NO-THREADS_Female-Threaded-Hex-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 scale=0.001 0.001 0.001
- link 94868A713_NO-THREADS_Female-Threaded-Hex-Standoff-5: geometry collision mesh filename=meshes/reauthored/94868A713_NO-THREADS_Female-Threaded-Hex-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 scale=0.001 0.001 0.001; visual mesh filename=meshes/reauthored/94868A713_NO-THREADS_Female-Threaded-Hex-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 scale=0.001 0.001 0.001
- link Battery---Battery-5.2-Ah-DC5521-Plug-v2: geometry collision mesh filename=meshes/reauthored/Battery---Battery-5.2-Ah-DC5521-Plug-v2.s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 scale=0.001 0.001 0.001; visual mesh filename=meshes/reauthored/Battery---Battery-5.2-Ah-DC5521-Plug-v2.s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 scale=0.001 0.001 0.001
- link Camera-Model-v3: geometry collision mesh filename=meshes/reauthored/Camera-Model-v3.stl scale=0.001 0.001 0.001; visual mesh filename=meshes/reauthored/Camera-Model-v3.stl scale=0.001 0.001 0.001
- link Camera-Mount-v8: geometry collision mesh filename=meshes/reauthored/Camera-Mount-v8.stl scale=0.001 0.001 0.001; visual mesh filename=meshes/reauthored/Camera-Mount-v8.stl scale=0.001 0.001 0.001
- link ST3215_Servo_Motor-v1: geometry collision mesh filename=meshes/reauthored/ST3215_Servo_Motor-v1.stl scale=0.001 0.001 0.001; visual mesh filename=meshes/reauthored/ST3215_Servo_Motor-v1.stl scale=0.001 0.001 0.001
- link ST3215_Servo_Motor-v1-1: geometry collision mesh filename=meshes/reauthored/ST3215_Servo_Motor-v1-1.stl scale=0.001 0.001 0.001; visual mesh filename=meshes/reauthored/ST3215_Servo_Motor-v1-1.stl scale=0.001 0.001 0.001
- link ST3215_Servo_Motor-v1-2: geometry collision mesh filename=meshes/reauthored/ST3215_Servo_Motor-v1-2.stl scale=0.001 0.001 0.001; visual mesh filename=meshes/reauthored/ST3215_Servo_Motor-v1-2.stl scale=0.001 0.001 0.001
- link base_plate_layer1-v5: geometry collision mesh filename=meshes/reauthored/base_plate_layer1-v5.stl scale=0.001 0.001 0.001; visual mesh filename=meshes/reauthored/base_plate_layer1-v5.stl scale=0.001 0.001 0.001
- link base_plate_layer2-v3: geometry collision mesh filename=meshes/reauthored/base_plate_layer2-v3.stl scale=0.001 0.001 0.001; visual mesh filename=meshes/reauthored/base_plate_layer2-v3.stl scale=0.001 0.001 0.001
- link drive_motor_mount-v11: geometry collision mesh filename=meshes/reauthored/drive_motor_mount-v11.stl scale=0.001 0.001 0.001; visual mesh filename=meshes/reauthored/drive_motor_mount-v11.stl scale=0.001 0.001 0.001
- link drive_motor_mount-v11-1: geometry collision mesh filename=meshes/reauthored/drive_motor_mount-v11-1.stl scale=0.001 0.001 0.001; visual mesh filename=meshes/reauthored/drive_motor_mount-v11-1.stl scale=0.001 0.001 0.001
- link drive_motor_mount-v11-2: geometry collision mesh filename=meshes/reauthored/drive_motor_mount-v11-2.stl scale=0.001 0.001 0.001; visual mesh filename=meshes/reauthored/drive_motor_mount-v11-2.stl scale=0.001 0.001 0.001
- link lipo_battery_mount-v3: geometry collision mesh filename=meshes/reauthored/lipo_battery_mount-v3.stl scale=0.001 0.001 0.001; visual mesh filename=meshes/reauthored/lipo_battery_mount-v3.stl scale=0.001 0.001 0.001
- link omni_wheel_mount-v5: geometry collision mesh filename=meshes/reauthored/omni_wheel_mount-v5.stl scale=0.001 0.001 0.001; visual mesh filename=meshes/reauthored/omni_wheel_mount-v5.stl scale=0.001 0.001 0.001
- link omni_wheel_mount-v5-1: geometry collision mesh filename=meshes/reauthored/omni_wheel_mount-v5-1.stl scale=0.001 0.001 0.001; visual mesh filename=meshes/reauthored/omni_wheel_mount-v5-1.stl scale=0.001 0.001 0.001
- link omni_wheel_mount-v5-2: geometry collision mesh filename=meshes/reauthored/omni_wheel_mount-v5-2.stl scale=0.001 0.001 0.001; visual mesh filename=meshes/reauthored/omni_wheel_mount-v5-2.stl scale=0.001 0.001 0.001
- link servo_controller_mount-v3: geometry collision mesh filename=meshes/reauthored/servo_controller_mount-v3.stl scale=0.001 0.001 0.001; visual mesh filename=meshes/reauthored/servo_controller_mount-v3.stl scale=0.001 0.001 0.001
- link so101_wrist_link: geometry collision mesh filename=meshes/so101/native_wrist_flex.stl; collision mesh filename=meshes/so101/sts3215_03a_no_horn_v1.stl
Joints:
- removed joint Bottom-V2-v3_Rigid-24
- removed joint base_plate_layer2-v3_Rigid-22
- added joint astra_pro_compact_mount_joint: type fixed, parent base_plate_layer2-v3, child astra_pro_compact_mount, origin xyz=-0.09 -0.04 0.007 rpy=0.0 0.0 2.0344439357957027
- added joint ld06_body_mount: type fixed, parent robotskin_lidar_mount, child ld06_body, origin xyz=0.02 -0.005 0.012 rpy=0 0 0
- added joint robotskin_lidar_mount_joint: type fixed, parent base_plate_layer2-v3, child robotskin_lidar_mount, origin xyz=0.0 -0.115 0.007 rpy=0.0 0.0 -1.5707963267948966
- added joint rpi5_table_joint: type fixed, parent rpi5_through_plate, child rpi5_table, origin xyz=0.0 0.0 0.004 rpy=0 0 0
- added joint rpi5_through_plate_joint: type fixed, parent base_plate_layer2-v3, child rpi5_through_plate, origin xyz=0.125 -0.075 0.007 rpy=0.0 0.0 -1.5707963267948966
- added joint rpi5_usb_carrier_joint: type fixed, parent rpi5_through_plate, child rpi5_usb_carrier, origin xyz=0.0 0.0 0.004 rpy=0 0 0
- joint 94868A713_NO-THREADS_Female-Threaded-Hex-Standoff_Rigid-21: origin xyz=0.0 0.0 -0.05 rpy=3.141592653589793 -0.0 0.0 -> xyz=0.06 0.08 -0.05 rpy=3.141592653589793 -0.0 0.0
- joint base_plate_layer1-v5_Rigid-20: origin xyz=0.0 0.0 0.0 rpy=3.141592653589793 -0.0 0.0 -> xyz=-0.06 0.08 0 rpy=3.141592653589793 -0.0 0.0
- joint base_plate_layer1-v5_Rigid-30: origin xyz=0.02 -0.1 0.0 rpy=3.141592653589793 -0.0 0.0 -> xyz=0.06 -0.08 0 rpy=3.141592653589793 -0.0 0.0
- joint base_plate_layer1-v5_Rigid-31: origin xyz=0.07660254 0.06732051 0.0 rpy=3.141592653589793 -0.0 0.0 -> xyz=0.06 0.08 0 rpy=3.141592653589793 -0.0 0.0
- joint base_plate_layer1-v5_Rigid-32: origin xyz=-0.09660254 0.032679490000000005 0.0 rpy=3.141592653589793 -0.0 0.0 -> xyz=-0.06 -0.08 0 rpy=3.141592653589793 -0.0 0.0
- joint base_plate_layer1-v5_Rigid-69: origin xyz=0.1 -0.02 0.0 rpy=3.141592653589793 -0.0 0.0 -> xyz=0.1 0 0 rpy=3.141592653589793 -0.0 0.0
- joint base_plate_layer1-v5_Rigid-70: origin xyz=-0.1 -0.02 0.0 rpy=3.141592653589793 -0.0 0.0 -> xyz=-0.1 0 0 rpy=3.141592653589793 -0.0 0.0
- joint base_plate_layer1-v5_baseplate2bottom_mount: origin xyz=-0.02 -0.1 0.0 rpy=3.141592653589793 -0.0 0.0 -> xyz=0.02375 -0.06895 0 rpy=1.57079632679 0 -1.57079632679
- joint base_plate_layer1-v5_baseplate2left_mount: origin xyz=-0.05928203 0.057320510000000005 0.0 rpy=3.141592653589793 -0.0 0.0 -> xyz=-0.0715874515909 0.0139068966601 0 rpy=1.57079632679 2.77555756156e-17 2.61799387799
- joint base_plate_layer1-v5_baseplate2right_mount: origin xyz=0.07928203 0.022679490000000004 0.0 rpy=0.0 -0.0 0.0 -> xyz=0.0478374515909 0.0550431033399 0 rpy=1.57079632679 0 0.523598775598
- joint drive_motor_mount-v11-1_Rigid-35: origin xyz=-0.007786400000000002 -0.018513550000000004 0.0076100000000000004 rpy=-7.401486830834375e-17 -1.5707963267948966 0 -> xyz=0.00555000203031 0.0429865595601 0.0339999998126 rpy=-3.66519142919 1.57079632679 0
- joint drive_motor_mount-v11-2_Rigid-2: origin xyz=-0.01214 -0.015999999999999997 -0.0076100000000000004 rpy=3.141592653589793 1.5707963267948966 0 -> xyz=0.00555000019073 0.0429865544308 0.0339999998126 rpy=-1.57079632679 1.57079632679 0
- joint drive_motor_mount-v11_Rigid-39: origin xyz=0.019926399999999997 -0.0025135499999999933 -0.0076100000000000004 rpy=3.141592653589793 1.5707963267948966 0 -> xyz=0.00555000555268 0.0429865554023 0.0339999998126 rpy=-5.75958653158 1.57079632679 0
- joint so101_mount: origin xyz=0.0388353 0.06714801 0.007 rpy=0 0 3.14159 -> xyz=-8.90955448261e-08 0.0283127100002 0.00699999999992 rpy=-2.65358979335e-06 -7.04151787872e-12 1.57079
