Commit message: Add deterministic FreeCAD robot export

File: URDF/LeKiwi.urdf.xacro (robot description, xacro)
@@ -6,5 +6,5 @@
             <origin xyz="-4.730687660675253e-15 -2.7155537377808555e-05 -0.0035000000000000005" rpy="0.0 0.0 0.0" />
             <mass value="1.9468624348344596" />
-            <inertia ixx="0.005637109888809055" iyy="0.005628440956780792" izz="0.0112496514690387" ixy="1.3447333053523504e-16" iyz="2.6469779601696886e-23" ixz="1.7848833522297417e-20" />
+            <inertia ixx="0.005637109888809055" iyy="0.005628440956780792" izz="0.0112496514690387" ixy="1.3447333053523504e-16" ixz="1.7848833522297417e-20" iyz="2.6469779601696886e-23" />
         </inertial>
         <visual name="base_plate_layer1-v5_visual">
@@ -25,5 +25,5 @@
             <origin xyz="-0.0005387977877578853 0.00013596517365616734 -0.0031122813365712966" rpy="0.0 -0.0 0.0" />
             <mass value="0.047242276734470956" />
-            <inertia ixx="5.0825527819301506e-06" iyy="4.311179042786683e-06" izz="8.973045405784286e-06" ixy="-1.350766273806132e-08" iyz="3.9985254125769694e-08" ixz="-1.2930640441004792e-07" />
+            <inertia ixx="5.0825527819301506e-06" iyy="4.311179042786683e-06" izz="8.973045405784286e-06" ixy="-1.350766273806132e-08" ixz="-1.2930640441004792e-07" iyz="3.9985254125769694e-08" />
         </inertial>
         <visual name="drive_motor_mount-v11-2_visual">
@@ -44,5 +44,5 @@
             <origin xyz="0.010251219185305343 -0.016877183343657672 -0.021914257028179583" rpy="0.0 -0.0 0.0" />
             <mass value="0.0658962961901927" />
-            <inertia ixx="1.8215748982019337e-05" iyy="1.391369165568997e-05" izz="1.030090838794644e-05" ixy="-8.885501451912254e-10" iyz="-1.195158171269568e-07" ixz="-1.7998869276666056e-09" />
+            <inertia ixx="1.8215748982019337e-05" iyy="1.391369165568997e-05" izz="1.030090838794644e-05" ixy="-8.885501451912254e-10" ixz="-1.7998869276666056e-09" iyz="-1.195158171269568e-07" />
         </inertial>
         <visual name="ST3215_Servo_Motor-v1-2_visual">
@@ -63,5 +63,5 @@
             <origin xyz="-9.805110055688405e-08 0.015875012090586064 -9.143534264177689e-08" rpy="0.0 -0.0 0.0" />
             <mass value="1.3542854082324305" />
-            <inertia ixx="0.0010936167993003225" iyy="0.0018798127501507863" izz="0.0010936140861738455" ixy="-4.1677764986761383e-10" iyz="8.101180750536008e-12" ixz="-6.83978047246436e-09" />
+            <inertia ixx="0.0010936167993003225" iyy="0.0018798127501507863" izz="0.0010936140861738455" ixy="-4.1677764986761383e-10" ixz="-6.83978047246436e-09" iyz="8.101180750536008e-12" />
         </inertial>
         <visual name="4-Omni-Directional-Wheel_Single_Body-v1-2_visual">
@@ -82,5 +82,5 @@
             <origin xyz="5.9743256737576635e-09 -5.0148034724806225e-09 -0.005522899140934374" rpy="0.0 -0.0 0.0" />
             <mass value="0.1235708646349694" />
-            <inertia ixx="1.78648151778313e-05" iyy="1.7864798695374842e-05" izz="3.26402691752235e-05" ixy="3.1863413372475765e-12" iyz="-4.243561882097402e-14" ixz="4.731358839058734e-14" />
+            <inertia ixx="1.78648151778313e-05" iyy="1.7864798695374842e-05" izz="3.26402691752235e-05" ixy="3.1863413372475765e-12" ixz="4.731358839058734e-14" iyz="-4.243561882097402e-14" />
         </inertial>
         <visual name="omni_wheel_mount-v5-2_visual">
@@ -101,5 +101,5 @@
             <origin xyz="0.00038715049105024767 -0.0003986280605619008 0.0031122813365712966" rpy="0.0 -0.0 0.0" />
             <mass value="0.047242276734470956" />
-            <inertia ixx="4.515720456649471e-06" iyy="4.8780113680673386e-06" izz="8.973045405784395e-06" ixy="-3.4076845832425005e-07" iyz="9.199000402824292e-08" ixz="-9.928144805471037e-08" />
+            <inertia ixx="4.515720456649471e-06" iyy="4.8780113680673386e-06" izz="8.973045405784395e-06" ixy="-3.4076845832425005e-07" ixz="-9.928144805471037e-08" iyz="9.199000402824292e-08" />
         </inertial>
         <visual name="drive_motor_mount-v11-1_visual">
@@ -120,5 +120,5 @@
             <origin xyz="0.01025121918530536 0.027816898485662264 -0.00435175717107704" rpy="0.0 -0.0 0.0" />
             <mass value="0.0658962961901927" />
-            <inertia ixx="1.82157489820195e-05" iyy="1.1100600471096564e-05" izz="1.3113999572540226e-05" ixy="2.0030228758654146e-09" iyz="-1.504623135553104e-06" ixz="1.3043646559715847e-10" />
+            <inertia ixx="1.82157489820195e-05" iyy="1.1100600471096564e-05" izz="1.3113999572540226e-05" ixy="2.0030228758654146e-09" ixz="1.3043646559715847e-10" iyz="-1.504623135553104e-06" />
         </inertial>
         <visual name="ST3215_Servo_Motor-v1-1_visual">
@@ -139,5 +139,5 @@
             <origin xyz="0.004782968825905343 5.966875074037148e-09 0.0027614494161754166" rpy="0.0 -0.0 0.0" />
             <mass value="0.1235708646349694" />
-            <inertia ixx="2.8946401592011724e-05" iyy="1.7864815177831735e-05" izz="2.155866627858642e-05" ixy="1.5521959531496902e-12" iyz="-2.7831093278498503e-12" ixz="6.397966372990203e-06" />
+            <inertia ixx="2.8946401592011724e-05" iyy="1.7864815177831735e-05" izz="2.155866627858642e-05" ixy="1.5521959531496902e-12" ixz="6.397966372990203e-06" iyz="-2.7831093278498503e-12" />
         </inertial>
         <visual name="omni_wheel_mount-v5-1_visual">
@@ -158,5 +158,5 @@
             <origin xyz="0.01374810955311503 -0.007937600014431929 -7.105207897817323e-08" rpy="0.0 -0.0 0.0" />
             <mass value="1.3542854082324305" />
-            <inertia ixx="0.0016832621879788534" iyy="0.0012901614102005313" izz="0.0010936200374455259" ixy="-0.0003404354598931583" iyz="-4.340089721204671e-09" ixz="-2.9730281413814508e-09" />
+            <inertia ixx="0.0016832621879788534" iyy="0.0012901614102005313" izz="0.0010936200374455259" ixy="-0.0003404354598931583" ixz="-2.9730281413814508e-09" iyz="-4.340089721204671e-09" />
         </inertial>
         <visual name="4-Omni-Directional-Wheel_Single_Body-v1-1_visual">
@@ -177,5 +177,5 @@
             <origin xyz="0.00015164729670767764 -0.0005345932342180682 -0.003112281336571299" rpy="0.0 -0.0 0.0" />
             <mass value="0.047242276734470956" />
-            <inertia ixx="4.492324498495657e-06" iyy="4.901407326221227e-06" izz="8.973045405784395e-06" ixy="-3.2726079558618873e-07" iyz="-1.319752581540088e-07" ixz="3.002495635533459e-08" />
+            <inertia ixx="4.492324498495657e-06" iyy="4.901407326221227e-06" izz="8.973045405784395e-06" ixy="-3.2726079558618873e-07" ixz="3.002495635533459e-08" iyz="-1.319752581540088e-07" />
         </inertial>
         <visual name="drive_motor_mount-v11_visual">
@@ -196,5 +196,5 @@
             <origin xyz="0.010251219185305386 -0.010539715142004517 0.02557319387622896" rpy="-6.077163357286271e-64 -0.0 0.0" />
             <mass value="0.0658962961901927" />
-            <inertia ixx="1.8215748982019662e-05" iyy="1.1307607938668487e-05" izz="1.2906992104968112e-05" ixy="-1.1144727307283995e-09" iyz="1.6241389526799929e-06" ixz="1.6694504620406482e-09" />
+            <inertia ixx="1.8215748982019662e-05" iyy="1.1307607938668487e-05" izz="1.2906992104968112e-05" ixy="-1.1144727307283995e-09" ixz="1.6694504620406482e-09" iyz="1.6241389526799929e-06" />
         </inertial>
         <visual name="ST3215_Servo_Motor-v1_visual">
@@ -215,5 +215,5 @@
             <origin xyz="-0.00478297352513172 5.966875045171349e-09 0.002761449724759064" rpy="0.0 -0.0 0.0" />
             <mass value="0.1235708646349694" />
-            <inertia ixx="2.8946401518511002e-05" iyy="1.7864815177831735e-05" izz="2.155866635208752e-05" ixy="1.634145428567116e-12" iyz="2.7357957614821196e-12" ixz="-6.397966415425984e-06" />
+            <inertia ixx="2.8946401518511002e-05" iyy="1.7864815177831735e-05" izz="2.155866635208752e-05" ixy="1.634145428567116e-12" ixz="-6.397966415425984e-06" iyz="2.7357957614821196e-12" />
         </inertial>
         <visual name="omni_wheel_mount-v5_visual">
@@ -234,5 +234,5 @@
             <origin xyz="-0.013748211804798878 -0.007937431357202592 -9.805855119449092e-08" rpy="0.0 1.0947644252537633e-47 6.865185903486632e-63" />
             <mass value="1.3542854082324305" />
-            <inertia ixx="0.00168326307714072" iyy="0.0012901637591839067" izz="0.001093616799300322" ixy="0.00034043401176330265" iyz="6.131812470911233e-09" ixz="-3.0589502042488444e-09" />
+            <inertia ixx="0.00168326307714072" iyy="0.0012901637591839067" izz="0.001093616799300322" ixy="0.00034043401176330265" ixz="-3.0589502042488444e-09" iyz="6.131812470911233e-09" />
         </inertial>
         <visual name="4-Omni-Directional-Wheel_Single_Body-v1_visual">
@@ -253,5 +253,5 @@
             <origin xyz="-2.072913100236695e-30 -3.385736135896877e-14 0.0031621761491414137" rpy="0.0 -0.0 0.0" />
             <mass value="0.12559881449596652" />
-            <inertia ixx="3.9342162518597853e-05" iyy="2.2687082259147483e-05" izz="6.101873120031777e-05" ixy="-1.0198295364639013e-21" iyz="-1.1248597539537109e-18" ixz="-2.788880237858462e-21" />
+            <inertia ixx="3.9342162518597853e-05" iyy="2.2687082259147483e-05" izz="6.101873120031777e-05" ixy="-1.0198295364639013e-21" ixz="-2.788880237858462e-21" iyz="-1.1248597539537109e-18" />
         </inertial>
         <visual name="servo_controller_mount-v3_visual">
@@ -272,5 +272,5 @@
             <origin xyz="-0.008318729060206734 -4.4408920985006264e-17 -0.0046380028574369405" rpy="0.0 -0.0 0.0" />
             <mass value="0.2984320446179905" />
-            <inertia ixx="0.00012005856115871003" iyy="0.0001714977017617139" izz="0.0002832588139475423" ixy="-8.673617379884035e-19" iyz="1.3552527156068805e-20" ixz="3.436962366808516e-06" />
+            <inertia ixx="0.00012005856115871003" iyy="0.0001714977017617139" izz="0.0002832588139475423" ixy="-8.673617379884035e-19" ixz="3.436962366808516e-06" iyz="1.3552527156068805e-20" />
         </inertial>
         <visual name="lipo_battery_mount-v3_visual">
@@ -291,5 +291,5 @@
             <origin xyz="-7.797576827959673e-05 -8.300646300726023e-05 0.020000000000000004" rpy="0.0 -0.0 0.0" />
             <mass value="1.2215469988184764" />
-            <inertia ixx="0.00047597821218279624" iyy="0.00065975897252246" izz="0.0008162228074590446" ixy="-3.1353787147811365e-06" iyz="1.3010426069826053e-18" ixz="-8.673617379884035e-19" />
+            <inertia ixx="0.00047597821218279624" iyy="0.00065975897252246" izz="0.0008162228074590446" ixy="-3.1353787147811365e-06" ixz="-8.673617379884035e-19" iyz="1.3010426069826053e-18" />
         </inertial>
         <visual name="Battery---Battery-5.2-Ah-DC5521-Plug-v2_visual">
@@ -310,5 +310,5 @@
             <origin xyz="2.1864399078485972e-14 1.2010287410706806e-09 -0.02499999330297986" rpy="0.0 -0.0 0.0" />
             <mass value="0.006150070863406618" />
-            <inertia ixx="1.0965196650850464e-06" iyy="1.096519654894581e-06" izz="1.837396493115053e-08" ixy="-3.0209076389532564e-20" iyz="-9.149560120561933e-14" ixz="-2.6974127807751317e-18" />
+            <inertia ixx="1.0965196650850464e-06" iyy="1.096519654894581e-06" izz="1.837396493115053e-08" ixy="-3.0209076389532564e-20" ixz="-2.6974127807751317e-18" iyz="-9.149560120561933e-14" />
         </inertial>
         <visual name="94868A713_NO-THREADS_Female-Threaded-Hex-Standoff_visual">
@@ -329,5 +329,5 @@
             <origin xyz="1.4406667835883843e-14 -0.000737848116891558 0.0034999999999999966" rpy="0.0 -0.0 0.0" />
             <mass value="1.9153836917607525" />
-            <inertia ixx="0.005568248812566009" iyy="0.00562277090534615" izz="0.01117537741776278" ixy="-1.3825833742235038e-15" iyz="1.3552527156068805e-20" ixz="1.6063950170089246e-19" />
+            <inertia ixx="0.005568248812566009" iyy="0.00562277090534615" izz="0.01117537741776278" ixy="-1.3825833742235038e-15" ixz="1.6063950170089246e-19" iyz="1.3552527156068805e-20" />
         </inertial>
         <visual name="base_plate_layer2-v3_visual">
@@ -348,5 +348,5 @@
             <origin xyz="0.021623799145011228 0.034248555702746215 0.002860022373659428" rpy="0.0 -0.0 0.0" />
             <mass value="0.14588862570926195" />
-            <inertia ixx="5.861212367196979e-05" iyy="0.00012648590487769422" izz="0.0001820968398762769" ixy="1.504419769130789e-06" iyz="7.708271472892277e-07" ixz="-2.5907710844293995e-06" />
+            <inertia ixx="5.861212367196979e-05" iyy="0.00012648590487769422" izz="0.0001820968398762769" ixy="1.504419769130789e-06" ixz="-2.5907710844293995e-06" iyz="7.708271472892277e-07" />
         </inertial>
         <visual name="Bottom-V2-v3_visual">
@@ -367,5 +367,5 @@
             <origin xyz="0.00394392416615524 -0.00045096335632409 0.021552698750372336" rpy="0.0 -0.0 0.0" />
             <mass value="0.1256590419653392" />
-            <inertia ixx="5.8982381320791524e-05" iyy="0.00013338786905954623" izz="0.00018586375094365218" ixy="-1.6170683703386755e-07" iyz="5.073018525688332e-07" ixz="2.7949770042390678e-06" />
+            <inertia ixx="5.8982381320791524e-05" iyy="0.00013338786905954623" izz="0.00018586375094365218" ixy="-1.6170683703386755e-07" ixz="2.7949770042390678e-06" iyz="5.073018525688332e-07" />
         </inertial>
         <visual name="Top-V2-v2_visual">
@@ -386,5 +386,5 @@
             <origin xyz="-0.019889007343132665 0.003162253231103023 0.020248493842242046" rpy="0.0 -0.0 0.0" />
             <mass value="0.09265469509875414" />
-            <inertia ixx="1.7978739433416715e-05" iyy="3.514579199775795e-05" izz="1.872943107726426e-05" ixy="2.2659313403750657e-08" iyz="1.493014354660236e-06" ixz="-1.7551355004084038e-07" />
+            <inertia ixx="1.7978739433416715e-05" iyy="3.514579199775795e-05" izz="1.872943107726426e-05" ixy="2.2659313403750657e-08" ixz="-1.7551355004084038e-07" iyz="1.493014354660236e-06" />
         </inertial>
         <visual name="Camera-Mount-v8_visual">
@@ -405,5 +405,5 @@
             <origin xyz="-0.01552129548236823 0.006733132771749837 -0.011599583774026805" rpy="0.0 2.7755575615628914e-17 0.0" />
             <mass value="0.039920058315088616" />
-            <inertia ixx="5.3846132096854386e-06" iyy="7.612080863465678e-06" izz="5.20250984027362e-06" ixy="3.6969144888008537e-07" iyz="-9.014266851093004e-08" ixz="3.317962541199677e-08" />
+            <inertia ixx="5.3846132096854386e-06" iyy="7.612080863465678e-06" izz="5.20250984027362e-06" ixy="3.6969144888008537e-07" ixz="3.317962541199677e-08" iyz="-9.014266851093004e-08" />
         </inertial>
         <visual name="Camera-Model-v3_visual">
@@ -424,5 +424,5 @@
             <origin xyz="-0.03999704723368316 -0.03974905501648025 0.021865523723532104" rpy="0.0 -0.0 0.0" />
             <mass value="1.2829039880853146" />
-            <inertia ixx="0.0013599465686859134" iyy="0.0015570925522625356" izz="0.0017754186964794674" ixy="-2.7674912025085476e-08" iyz="0.00024876935781550404" ixz="-1.4799628966957228e-07" />
+            <inertia ixx="0.0013599465686859134" iyy="0.0015570925522625356" izz="0.0017754186964794674" ixy="-2.7674912025085476e-08" ixz="-1.4799628966957228e-07" iyz="0.00024876935781550404" />
         </inertial>
         <visual name="Base_08q-v1_visual">
@@ -443,5 +443,5 @@
             <origin xyz="-0.0036802122213187593 -0.0036094977362838856 6.824776544718247e-06" rpy="0.0 -0.0 0.0" />
             <mass value="0.07141322001638221" />
-            <inertia ixx="1.5714974230074772e-05" iyy="1.571497423007476e-05" izz="1.3312770357058572e-05" ixy="6.4527910706321766e-06" iyz="1.5349694469765155e-10" ixz="1.534969447374064e-10" />
+            <inertia ixx="1.5714974230074772e-05" iyy="1.571497423007476e-05" izz="1.3312770357058572e-05" ixy="6.4527910706321766e-06" ixz="1.534969447374064e-10" iyz="1.5349694469765155e-10" />
         </inertial>
         <visual name="WaveShare_Mounting_Plate_01d-v1_visual">
@@ -462,5 +462,5 @@
             <origin xyz="0.00027157225787806426 -0.03155586567874573 0.009540449649933115" rpy="4.3790577010150533e-47 4.379057701015054e-47 -1.5557538194652858e-61" />
             <mass value="0.5385469320676795" />
-            <inertia ixx="0.00037498929247645185" iyy="0.00034052316913093367" izz="0.00015416122792210035" ixy="-6.375305991054909e-07" iyz="-3.6006983324524115e-05" ixz="3.4882693251635207e-06" />
+            <inertia ixx="0.00037498929247645185" iyy="0.00034052316913093367" izz="0.00015416122792210035" ixy="-6.375305991054909e-07" ixz="3.4882693251635207e-06" iyz="-3.6006983324524115e-05" />
         </inertial>
         <visual name="Rotation_Pitch_08i-v1_visual">
@@ -481,5 +481,5 @@
             <origin xyz="-0.010249997314858655 0.016027064924721765 -0.019999026815617257" rpy="0.0 -0.0 0.0" />
             <mass value="0.2843033831904074" />
-            <inertia ixx="7.348827769135388e-05" iyy="6.153681935695018e-05" izz="3.972527876478296e-05" ixy="-2.948942387958768e-14" iyz="5.568928366529984e-07" ixz="4.0140055866208044e-14" />
+            <inertia ixx="7.348827769135388e-05" iyy="6.153681935695018e-05" izz="3.972527876478296e-05" ixy="-2.948942387958768e-14" ixz="4.0140055866208044e-14" iyz="5.568928366529984e-07" />
         </inertial>
         <visual name="STS3215_03a-v1_visual">
@@ -500,5 +500,5 @@
             <origin xyz="-0.023249790543467236 0.009494231975835899 0.002658209837920218" rpy="0.0 -0.0 0.0" />
             <mass value="0.10853073755546007" />
-            <inertia ixx="2.6819408873440288e-05" iyy="4.591982320177254e-05" izz="5.824324969726431e-05" ixy="-1.7483214372584268e-07" iyz="-5.297613839098936e-08" ixz="-1.9180973510858863e-07" />
+            <inertia ixx="2.6819408873440288e-05" iyy="4.591982320177254e-05" izz="5.824324969726431e-05" ixy="-1.7483214372584268e-07" ixz="-1.9180973510858863e-07" iyz="-5.297613839098936e-08" />
         </inertial>
         <visual name="SO_ARM100_08k_Asym_Mirror_Clip-v1_visual">
@@ -519,5 +519,5 @@
             <origin xyz="2.6917174546039143e-09 -0.0010740097666846627 -7.475931163014593e-10" rpy="0.0 -0.0 0.0" />
             <mass value="0.00454511487954422" />
-            <inertia ixx="1.2518150597416012e-07" iyy="2.464408524633815e-07" izz="1.2518150393394235e-07" ixy="-1.283788438507426e-19" iyz="0.0" ixz="8.715254501525044e-23" />
+            <inertia ixx="1.2518150597416012e-07" iyy="2.464408524633815e-07" izz="1.2518150393394235e-07" ixy="-1.283788438507426e-19" ixz="8.715254501525044e-23" iyz="0.0" />
         </inertial>
         <visual name="Passive_Horn_01-v1_visual">
@@ -538,5 +538,5 @@
             <origin xyz="0.0160270676166179 0.010250000754348055 -0.01999902756321033" rpy="0.0 -0.0 0.0" />
             <mass value="0.2843033831904074" />
-            <inertia ixx="6.153681935694953e-05" iyy="7.348827769135171e-05" izz="3.972527876478253e-05" ixy="2.948943437265658e-14" iyz="-4.013890531409639e-14" ixz="5.568928366528663e-07" />
+            <inertia ixx="6.153681935694953e-05" iyy="7.348827769135171e-05" izz="3.972527876478253e-05" ixy="2.948943437265658e-14" ixz="5.568928366528663e-07" iyz="-4.013890531409639e-14" />
         </inertial>
         <visual name="STS3215_03a-v1-1_visual">
@@ -557,5 +557,5 @@
             <origin xyz="-0.019699521396133086 -0.057761973340815856 -0.00542034076312131" rpy="0.0 -0.0 0.0" />
             <mass value="0.9906249126045027" />
-            <inertia ixx="0.001250627685357622" iyy="0.0004892267713729921" izz="0.0016228645319323214" ixy="8.068202927851326e-06" iyz="-0.00011683370128806429" ixz="1.3596898095040173e-06" />
+            <inertia ixx="0.001250627685357622" iyy="0.0004892267713729921" izz="0.0016228645319323214" ixy="8.068202927851326e-06" ixz="1.3596898095040173e-06" iyz="-0.00011683370128806429" />
         </inertial>
         <visual name="SO_ARM100_08k_116_Square-v1_visual">
@@ -576,5 +576,5 @@
             <origin xyz="0.016027067616617895 -0.011954028773405692 0.019029580609805842" rpy="0.0 -0.0 -1.9446922743316068e-62" />
             <mass value="0.2843033831904074" />
-            <inertia ixx="6.153681935695127e-05" iyy="7.323180978895463e-05" izz="3.9981746667182695e-05" ixy="4.853637943208478e-08" iyz="2.9314415785545002e-06" ixz="-5.547736938490272e-07" />
+            <inertia ixx="6.153681935695127e-05" iyy="7.323180978895463e-05" izz="3.9981746667182695e-05" ixy="4.853637943208478e-08" ixz="-5.547736938490272e-07" iyz="2.9314415785545002e-06" />
         </inertial>
         <visual name="STS3215_03a-v1-2_visual">
@@ -595,5 +595,5 @@
             <origin xyz="-0.01521487611614386 0.06115231912604866 0.010924244381939695" rpy="0.0 -0.0 0.0" />
             <mass value="0.8772447501056027" />
-            <inertia ixx="0.0009927953405503495" iyy="0.0003938875410144718" izz="0.0012139125572331573" ixy="0.00011404883978774629" iyz="-0.00015860294019953095" ixz="2.1130712730160653e-05" />
+            <inertia ixx="0.0009927953405503495" iyy="0.0003938875410144718" izz="0.0012139125572331573" ixy="0.00011404883978774629" ixz="2.1130712730160653e-05" iyz="-0.00015860294019953095" />
         </inertial>
         <visual name="SO_ARM100_08k_Mirror-v1_visual">
@@ -614,5 +614,5 @@
             <origin xyz="0.016027067616617773 -0.021475086668919854 0.006621488568077219" rpy="0.0 -0.0 0.0" />
             <mass value="0.2843033831904074" />
-            <inertia ixx="6.153681935695127e-05" iyy="4.074335774088658e-05" izz="7.247019871524764e-05" ixy="5.484323882535203e-07" iyz="-5.773812828266185e-06" ixz="9.670339719917652e-08" />
+            <inertia ixx="6.153681935695127e-05" iyy="4.074335774088658e-05" izz="7.247019871524764e-05" ixy="5.484323882535203e-07" ixz="9.670339719917652e-08" iyz="-5.773812828266185e-06" />
         </inertial>
         <visual name="STS3215_03a-v1-3_visual">
@@ -633,5 +633,5 @@
             <origin xyz="-0.016809778580177636 0.011102331354009483 -0.023929944943314147" rpy="0.0 -0.0 0.0" />
             <mass value="0.2392168278135931" />
-            <inertia ixx="0.00011529218614688731" iyy="0.00018638564430360945" izz="0.00013965599636815533" ixy="-2.876087303228392e-06" iyz="2.8346655089702376e-05" ixz="6.069085592614985e-06" />
+            <inertia ixx="0.00011529218614688731" iyy="0.00018638564430360945" izz="0.00013965599636815533" ixy="-2.876087303228392e-06" ixz="6.069085592614985e-06" iyz="2.8346655089702376e-05" />
         </inertial>
         <visual name="Wrist_Roll_Pitch_08i-v1_visual">
@@ -652,5 +652,5 @@
             <origin xyz="-0.015998302175323338 0.01584440444633293 -0.009724875472953585" rpy="0.0 -0.0 0.0" />
             <mass value="0.2799142523131049" />
-            <inertia ixx="3.834851845043938e-05" iyy="6.944931198304971e-05" izz="6.249728558243347e-05" ixy="-6.399687685208939e-07" iyz="4.1425511727094175e-06" ixz="1.3724175470711101e-06" />
+            <inertia ixx="3.834851845043938e-05" iyy="6.944931198304971e-05" izz="6.249728558243347e-05" ixy="-6.399687685208939e-07" ixz="1.3724175470711101e-06" iyz="4.1425511727094175e-06" />
         </inertial>
         <visual name="STS3215_03a_Wrist_Roll-v1_visual">
@@ -671,5 +671,5 @@
             <origin xyz="0.013763229636538839 0.011847838431604849 -0.02681060701774312" rpy="0.0 -0.0 0.0" />
             <mass value="0.44698022927880193" />
-            <inertia ixx="0.0003009649490412908" iyy="0.000302335224862029" izz="0.00019663017287168712" ixy="-2.7280550079654427e-05" iyz="6.471570024008629e-05" ixz="4.8752001162076285e-05" />
+            <inertia ixx="0.0003009649490412908" iyy="0.000302335224862029" izz="0.00019663017287168712" ixy="-2.7280550079654427e-05" ixz="4.8752001162076285e-05" iyz="6.471570024008629e-05" />
         </inertial>
         <visual name="Wrist_Roll_08c-v1_visual">
@@ -690,5 +690,5 @@
             <origin xyz="-0.01999902487131423 -0.01606298453944074 0.010193612482126984" rpy="0.0 -0.0 0.0" />
             <mass value="0.2843033831904074" />
-            <inertia ixx="3.972527876478296e-05" iyy="7.135367321426094e-05" izz="6.367142383404377e-05" ixy="-2.35353046222804e-07" iyz="4.577674103164314e-06" ixz="5.047163313676162e-07" />
+            <inertia ixx="3.972527876478296e-05" iyy="7.135367321426094e-05" izz="6.367142383404377e-05" ixy="-2.35353046222804e-07" ixz="5.047163313676162e-07" iyz="4.577674103164314e-06" />
         </inertial>
         <visual name="STS3215_03a-v1-4_visual">
@@ -709,5 +709,5 @@
             <origin xyz="0.0016198187276587506 0.031683055327891375 -0.018764632295228623" rpy="0.0 -0.0 1.0947644252537636e-47" />
             <mass value="0.1586808414280307" />
-            <inertia ixx="8.673205684445445e-05" iyy="6.319638527524501e-05" izz="3.0882476447698426e-05" ixy="-1.6959196471754863e-06" iyz="1.690507657065021e-05" ixz="3.83219457506011e-06" />
+            <inertia ixx="8.673205684445445e-05" iyy="6.319638527524501e-05" izz="3.0882476447698426e-05" ixy="-1.6959196471754863e-06" ixz="3.83219457506011e-06" iyz="1.690507657065021e-05" />
         </inertial>
         <visual name="Moving_Jaw_08d-v1_visual">
@@ -728,5 +728,5 @@
             <origin xyz="-0.012386670399303806 -0.0001931819643147037 0.033744611486572575" rpy="0.0 -0.0 0.0" />
             <mass value="0.14254654385043797" />
-            <inertia ixx="6.637825885912572e-05" iyy="9.286021404085985e-05" izz="2.9364578730897446e-05" ixy="-1.9686261197744952e-08" iyz="5.578936388252534e-07" ixz="-2.8501487566848823e-07" />
+            <inertia ixx="6.637825885912572e-05" iyy="9.286021404085985e-05" izz="2.9364578730897446e-05" ixy="-1.9686261197744952e-08" ixz="-2.8501487566848823e-07" iyz="5.578936388252534e-07" />
         </inertial>
         <visual name="Wrist-Camera-Mount-v11_visual">
@@ -747,5 +747,5 @@
             <origin xyz="2.1866952693017084e-14 1.201028743125221e-09 -0.02499999330297986" rpy="0.0 -0.0 0.0" />
             <mass value="0.006150070863406618" />
-            <inertia ixx="1.0965196650850456e-06" iyy="1.0965196548945862e-06" izz="1.837396493115063e-08" ixy="-2.879912020664621e-20" iyz="-9.149560026045249e-14" ixz="-2.6969529040576923e-18" />
+            <inertia ixx="1.0965196650850456e-06" iyy="1.0965196548945862e-06" izz="1.837396493115063e-08" ixy="-2.879912020664621e-20" ixz="-2.6969529040576923e-18" iyz="-9.149560026045249e-14" />
         </inertial>
         <visual name="94868A713_NO-THREADS_Female-Threaded-Hex-Standoff-1_visual">
@@ -766,5 +766,5 @@
             <origin xyz="2.1866952693017084e-14 1.201028743125221e-09 -0.02481596290467566" rpy="0.0 -0.0 0.0" />
             <mass value="0.006150070863406618" />
-            <inertia ixx="1.0965196650850456e-06" iyy="1.0965196548945997e-06" izz="1.837396493115063e-08" ixy="-3.3881317890172014e-20" iyz="-9.149560068396896e-14" ixz="-2.6969529040576923e-18" />
+            <inertia ixx="1.0965196650850456e-06" iyy="1.0965196548945997e-06" izz="1.837396493115063e-08" ixy="-3.3881317890172014e-20" ixz="-2.6969529040576923e-18" iyz="-9.149560068396896e-14" />
         </inertial>
         <visual name="94868A713_NO-THREADS_Female-Threaded-Hex-Standoff-2_visual">
@@ -785,5 +785,5 @@
             <origin xyz="0.00942672137716988 -0.014773756775059326 -0.01034538997402958" rpy="4.379057701015054e-47 -5.551115123125784e-17 0.0" />
             <mass value="0.039920058315088616" />
-            <inertia ixx="6.810843705690638e-06" iyy="5.386223522045076e-06" izz="6.002136685688621e-06" ixy="-3.1416649993652216e-07" iyz="-3.0173410406166294e-07" ixz="1.1161566006313797e-06" />
+            <inertia ixx="6.810843705690638e-06" iyy="5.386223522045076e-06" izz="6.002136685688621e-06" ixy="-3.1416649993652216e-07" ixz="1.1161566006313797e-06" iyz="-3.0173410406166294e-07" />
         </inertial>
         <visual name="Camera-Model-v3-1_visual">
@@ -804,5 +804,5 @@
             <origin xyz="-3.784219515523546e-10 -7.23282504999645e-10 -0.024999993302979855" rpy="0.0 -0.0 0.0" />
             <mass value="0.006150070863406618" />
-            <inertia ixx="1.0965196650850464e-06" iyy="1.0965196548945726e-06" izz="1.8373964931164182e-08" ixy="-2.710505431213761e-20" iyz="-9.149560110748543e-14" ixz="-2.6969529040576923e-18" />
+            <inertia ixx="1.0965196650850464e-06" iyy="1.0965196548945726e-06" izz="1.8373964931164182e-08" ixy="-2.710505431213761e-20" ixz="-2.6969529040576923e-18" iyz="-9.149560110748543e-14" />
         </inertial>
         <visual name="94868A713_NO-THREADS_Female-Threaded-Hex-Standoff-3_visual">
@@ -823,5 +823,5 @@
             <origin xyz="3.784657565120142e-10 3.1253399868091947e-09 -0.02499999330297986" rpy="0.0 -0.0 0.0" />
             <mass value="0.006150070863406618" />
-            <inertia ixx="1.0965196650850498e-06" iyy="1.0965196548945862e-06" izz="1.8373964931164182e-08" ixy="-2.710505431213761e-20" iyz="-9.149560110748543e-14" ixz="-2.6969529040576923e-18" />
+            <inertia ixx="1.0965196650850498e-06" iyy="1.0965196548945862e-06" izz="1.8373964931164182e-08" ixy="-2.710505431213761e-20" ixz="-2.6969529040576923e-18" iyz="-9.149560110748543e-14" />
         </inertial>
         <visual name="94868A713_NO-THREADS_Female-Threaded-Hex-Standoff-4_visual">
@@ -842,5 +842,5 @@
             <origin xyz="2.1862511800918584e-14 1.2010287342434368e-09 -0.02499999330297986" rpy="0.0 -0.0 0.0" />
             <mass value="0.006150070863406618" />
-            <inertia ixx="1.096519665085043e-06" iyy="1.0965196548945802e-06" izz="1.837396493115063e-08" ixy="-3.218725199566341e-20" iyz="-9.149560110748543e-14" ixz="-2.6969529040576923e-18" />
+            <inertia ixx="1.096519665085043e-06" iyy="1.0965196548945802e-06" izz="1.837396493115063e-08" ixy="-3.218725199566341e-20" ixz="-2.6969529040576923e-18" iyz="-9.149560110748543e-14" />
         </inertial>
         <visual name="94868A713_NO-THREADS_Female-Threaded-Hex-Standoff-5_visual">
