Commit message: Link editable base plates to robot export

File: URDF/LeKiwi.urdf.xacro (robot description, xacro)
@@ -9,13 +9,13 @@
         </inertial>
         <visual name="base_plate_layer1-v5_visual">
-            <origin xyz="0.0 0.0 0.0" rpy="0.0 0.0 0.0" />
-            <geometry>
-                <mesh filename="${mesh_dir}/base_plate_layer1-v5.stl" scale="0.001 0.001 0.001" />
+            <origin xyz="0 0 0" rpy="0 0 0" />
+            <geometry>
+                <mesh filename="${mesh_dir}/reauthored/base_plate_layer1-v5.stl" scale="0.001 0.001 0.001" />
             </geometry>
         </visual>
         <collision name="base_plate_layer1-v5_collision">
-            <origin xyz="0.0 0.0 0.0" rpy="0.0 0.0 0.0" />
-            <geometry>
-                <mesh filename="${mesh_dir}/base_plate_layer1-v5.stl" scale="0.001 0.001 0.001" />
+            <origin xyz="0 0 0" rpy="0 0 0" />
+            <geometry>
+                <mesh filename="${mesh_dir}/reauthored/base_plate_layer1-v5.stl" scale="0.001 0.001 0.001" />
             </geometry>
         </collision>
@@ -332,13 +332,13 @@
         </inertial>
         <visual name="base_plate_layer2-v3_visual">
-            <origin xyz="0.0 -6.430841866638185e-19 0.006999999999999993" rpy="0.0 -0.0 0.0" />
-            <geometry>
-                <mesh filename="${mesh_dir}/base_plate_layer2-v3.stl" scale="0.001 0.001 0.001" />
+            <origin xyz="0 0 0" rpy="0 0 0" />
+            <geometry>
+                <mesh filename="${mesh_dir}/reauthored/base_plate_layer2-v3.stl" scale="0.001 0.001 0.001" />
             </geometry>
         </visual>
         <collision name="base_plate_layer2-v3_collision">
-            <origin xyz="0.0 -6.430841866638185e-19 0.006999999999999993" rpy="0.0 -0.0 0.0" />
-            <geometry>
-                <mesh filename="${mesh_dir}/base_plate_layer2-v3.stl" scale="0.001 0.001 0.001" />
+            <origin xyz="0 0 0" rpy="0 0 0" />
+            <geometry>
+                <mesh filename="${mesh_dir}/reauthored/base_plate_layer2-v3.stl" scale="0.001 0.001 0.001" />
             </geometry>
         </collision>
