Commit message: Complete FreeCAD link migration

File: URDF/LeKiwi.urdf.xacro (robot description, xacro)
@@ -28,13 +28,13 @@
         </inertial>
         <visual name="drive_motor_mount-v11-2_visual">
-            <origin xyz="0.0 0.0 -0.0035000000000000005" rpy="3.141592653589793 -0.0 1.5707963267948966" />
-            <geometry>
-                <mesh filename="${mesh_dir}/drive_motor_mount-v11-2.stl" scale="0.001 0.001 0.001" />
+            <origin xyz="0 0 0" rpy="0 0 0" />
+            <geometry>
+                <mesh filename="${mesh_dir}/reauthored/drive_motor_mount-v11-2.stl" scale="0.001 0.001 0.001" />
             </geometry>
         </visual>
         <collision name="drive_motor_mount-v11-2_collision">
-            <origin xyz="0.0 0.0 -0.0035000000000000005" rpy="3.141592653589793 -0.0 1.5707963267948966" />
-            <geometry>
-                <mesh filename="${mesh_dir}/drive_motor_mount-v11-2.stl" scale="0.001 0.001 0.001" />
+            <origin xyz="0 0 0" rpy="0 0 0" />
+            <geometry>
+                <mesh filename="${mesh_dir}/reauthored/drive_motor_mount-v11-2.stl" scale="0.001 0.001 0.001" />
             </geometry>
         </collision>
@@ -47,13 +47,13 @@
         </inertial>
         <visual name="ST3215_Servo_Motor-v1-2_visual">
-            <origin xyz="0.010249999999999999 -0.025599999999999987 -0.007250000007450583" rpy="-3.141592653589793 -1.5707963267948966 0" />
-            <geometry>
-                <mesh filename="${mesh_dir}/ST3215_Servo_Motor-v1-2.stl" scale="0.001 0.001 0.001" />
+            <origin xyz="0 0 0" rpy="0 0 0" />
+            <geometry>
+                <mesh filename="${mesh_dir}/reauthored/ST3215_Servo_Motor-v1-2.stl" scale="0.001 0.001 0.001" />
             </geometry>
         </visual>
         <collision name="ST3215_Servo_Motor-v1-2_collision">
-            <origin xyz="0.010249999999999999 -0.025599999999999987 -0.007250000007450583" rpy="-3.141592653589793 -1.5707963267948966 0" />
-            <geometry>
-                <mesh filename="${mesh_dir}/ST3215_Servo_Motor-v1-2.stl" scale="0.001 0.001 0.001" />
+            <origin xyz="0 0 0" rpy="0 0 0" />
+            <geometry>
+                <mesh filename="${mesh_dir}/reauthored/ST3215_Servo_Motor-v1-2.stl" scale="0.001 0.001 0.001" />
             </geometry>
         </collision>
@@ -66,13 +66,13 @@
         </inertial>
         <visual name="4-Omni-Directional-Wheel_Single_Body-v1-2_visual">
-            <origin xyz="7.450578487500081e-12 0.015874999999999986 6.661338147750939e-18" rpy="1.5707963267948966 0.26179938779914924 -1.0046485565123013e-33" />
-            <geometry>
-                <mesh filename="${mesh_dir}/4-Omni-Directional-Wheel_Single_Body-v1-2.stl" scale="0.001 0.001 0.001" />
+            <origin xyz="0 0 0" rpy="0 0 0" />
+            <geometry>
+                <mesh filename="${mesh_dir}/reauthored/4-Omni-Directional-Wheel_Single_Body-v1-2.stl" scale="0.001 0.001 0.001" />
             </geometry>
         </visual>
         <collision name="4-Omni-Directional-Wheel_Single_Body-v1-2_collision">
-            <origin xyz="7.450578487500081e-12 0.015874999999999986 6.661338147750939e-18" rpy="1.5707963267948966 0.26179938779914924 -1.0046485565123013e-33" />
-            <geometry>
-                <mesh filename="${mesh_dir}/4-Omni-Directional-Wheel_Single_Body-v1-2.stl" scale="0.001 0.001 0.001" />
+            <origin xyz="0 0 0" rpy="0 0 0" />
+            <geometry>
+                <mesh filename="${mesh_dir}/reauthored/4-Omni-Directional-Wheel_Single_Body-v1-2.stl" scale="0.001 0.001 0.001" />
             </geometry>
         </collision>
@@ -85,13 +85,13 @@
         </inertial>
         <visual name="omni_wheel_mount-v5-2_visual">
-            <origin xyz="7.450581818169155e-12 2.220446049250313e-18 -0.005587499999999999" rpy="3.141592653589793 6.887535064975403e-49 1.8369701987210297e-16" />
-            <geometry>
-                <mesh filename="${mesh_dir}/omni_wheel_mount-v5-2.stl" scale="0.001 0.001 0.001" />
+            <origin xyz="0 0 0" rpy="0 0 0" />
+            <geometry>
+                <mesh filename="${mesh_dir}/reauthored/omni_wheel_mount-v5-2.stl" scale="0.001 0.001 0.001" />
             </geometry>
         </visual>
         <collision name="omni_wheel_mount-v5-2_collision">
-            <origin xyz="7.450581818169155e-12 2.220446049250313e-18 -0.005587499999999999" rpy="3.141592653589793 6.887535064975403e-49 1.8369701987210297e-16" />
-            <geometry>
-                <mesh filename="${mesh_dir}/omni_wheel_mount-v5-2.stl" scale="0.001 0.001 0.001" />
+            <origin xyz="0 0 0" rpy="0 0 0" />
+            <geometry>
+                <mesh filename="${mesh_dir}/reauthored/omni_wheel_mount-v5-2.stl" scale="0.001 0.001 0.001" />
             </geometry>
         </collision>
@@ -104,13 +104,13 @@
         </inertial>
         <visual name="drive_motor_mount-v11-1_visual">
-            <origin xyz="2.3027551065979426e-09 1.924311203715945e-09 0.0035000000000000005" rpy="0.0 -0.0 0.5235987755982988" />
-            <geometry>
-                <mesh filename="${mesh_dir}/drive_motor_mount-v11-1.stl" scale="0.001 0.001 0.001" />
+            <origin xyz="0 0 0" rpy="0 0 0" />
+            <geometry>
+                <mesh filename="${mesh_dir}/reauthored/drive_motor_mount-v11-1.stl" scale="0.001 0.001 0.001" />
             </geometry>
         </visual>
         <collision name="drive_motor_mount-v11-1_collision">
-            <origin xyz="2.3027551065979426e-09 1.924311203715945e-09 0.0035000000000000005" rpy="0.0 -0.0 0.5235987755982988" />
-            <geometry>
-                <mesh filename="${mesh_dir}/drive_motor_mount-v11-1.stl" scale="0.001 0.001 0.001" />
+            <origin xyz="0 0 0" rpy="0 0 0" />
+            <geometry>
+                <mesh filename="${mesh_dir}/reauthored/drive_motor_mount-v11-1.stl" scale="0.001 0.001 0.001" />
             </geometry>
         </collision>
@@ -123,13 +123,13 @@
         </inertial>
         <visual name="ST3215_Servo_Motor-v1-1_visual">
-            <origin xyz="0.010250000000000013 0.019478687706257793 -0.019238066498388086" rpy="-1.570796326794896 0.5235987755982991 -1.5707963267948968" />
-            <geometry>
-                <mesh filename="${mesh_dir}/ST3215_Servo_Motor-v1-1.stl" scale="0.001 0.001 0.001" />
+            <origin xyz="0 0 0" rpy="0 0 0" />
+            <geometry>
+                <mesh filename="${mesh_dir}/reauthored/ST3215_Servo_Motor-v1-1.stl" scale="0.001 0.001 0.001" />
             </geometry>
         </visual>
         <collision name="ST3215_Servo_Motor-v1-1_collision">
-            <origin xyz="0.010250000000000013 0.019478687706257793 -0.019238066498388086" rpy="-1.570796326794896 0.5235987755982991 -1.5707963267948968" />
-            <geometry>
-                <mesh filename="${mesh_dir}/ST3215_Servo_Motor-v1-1.stl" scale="0.001 0.001 0.001" />
+            <origin xyz="0 0 0" rpy="0 0 0" />
+            <geometry>
+                <mesh filename="${mesh_dir}/reauthored/ST3215_Servo_Motor-v1-1.stl" scale="0.001 0.001 0.001" />
             </geometry>
         </collision>
@@ -142,13 +142,13 @@
         </inertial>
         <visual name="omni_wheel_mount-v5-1_visual">
-            <origin xyz="0.004838917318364206 -1.7763568394002505e-17 0.002793745502761027" rpy="1.047197551196598 -1.1102230246251563e-16 1.5707963267948968" />
-            <geometry>
-                <mesh filename="${mesh_dir}/omni_wheel_mount-v5-1.stl" scale="0.001 0.001 0.001" />
+            <origin xyz="0 0 0" rpy="0 0 0" />
+            <geometry>
+                <mesh filename="${mesh_dir}/reauthored/omni_wheel_mount-v5-1.stl" scale="0.001 0.001 0.001" />
             </geometry>
         </visual>
         <collision name="omni_wheel_mount-v5-1_collision">
-            <origin xyz="0.004838917318364206 -1.7763568394002505e-17 0.002793745502761027" rpy="1.047197551196598 -1.1102230246251563e-16 1.5707963267948968" />
-            <geometry>
-                <mesh filename="${mesh_dir}/omni_wheel_mount-v5-1.stl" scale="0.001 0.001 0.001" />
+            <origin xyz="0 0 0" rpy="0 0 0" />
+            <geometry>
+                <mesh filename="${mesh_dir}/reauthored/omni_wheel_mount-v5-1.stl" scale="0.001 0.001 0.001" />
             </geometry>
         </collision>
@@ -161,13 +161,13 @@
         </inertial>
         <visual name="4-Omni-Directional-Wheel_Single_Body-v1-1_visual">
-            <origin xyz="0.013748155931950041 -0.007937495502761073 -2.2204460492503132e-17" rpy="-0.5235987755982988 -1.5707963267948963 0" />
-            <geometry>
-                <mesh filename="${mesh_dir}/4-Omni-Directional-Wheel_Single_Body-v1-1.stl" scale="0.001 0.001 0.001" />
+            <origin xyz="0 0 0" rpy="0 0 0" />
+            <geometry>
+                <mesh filename="${mesh_dir}/reauthored/4-Omni-Directional-Wheel_Single_Body-v1-1.stl" scale="0.001 0.001 0.001" />
             </geometry>
         </visual>
         <collision name="4-Omni-Directional-Wheel_Single_Body-v1-1_collision">
-            <origin xyz="0.013748155931950041 -0.007937495502761073 -2.2204460492503132e-17" rpy="-0.5235987755982988 -1.5707963267948963 0" />
-            <geometry>
-                <mesh filename="${mesh_dir}/4-Omni-Directional-Wheel_Single_Body-v1-1.stl" scale="0.001 0.001 0.001" />
+            <origin xyz="0 0 0" rpy="0 0 0" />
+            <geometry>
+                <mesh filename="${mesh_dir}/reauthored/4-Omni-Directional-Wheel_Single_Body-v1-1.stl" scale="0.001 0.001 0.001" />
             </geometry>
         </collision>
@@ -180,13 +180,13 @@
         </inertial>
         <visual name="drive_motor_mount-v11_visual">
-            <origin xyz="-2.3027550621890213e-09 1.9243111992750526e-09 -0.0035000000000000035" rpy="-3.141592653589793 -1.0340504353649803e-16 -2.6179938779914944" />
-            <geometry>
-                <mesh filename="${mesh_dir}/drive_motor_mount-v11.stl" scale="0.001 0.001 0.001" />
+            <origin xyz="0 0 0" rpy="0 0 0" />
+            <geometry>
+                <mesh filename="${mesh_dir}/reauthored/drive_motor_mount-v11.stl" scale="0.001 0.001 0.001" />
             </geometry>
         </visual>
         <collision name="drive_motor_mount-v11_collision">
-            <origin xyz="-2.3027550621890213e-09 1.9243111992750526e-09 -0.0035000000000000035" rpy="-3.141592653589793 -1.0340504353649803e-16 -2.6179938779914944" />
-            <geometry>
-                <mesh filename="${mesh_dir}/drive_motor_mount-v11.stl" scale="0.001 0.001 0.001" />
+            <origin xyz="0 0 0" rpy="0 0 0" />
+            <geometry>
+                <mesh filename="${mesh_dir}/reauthored/drive_motor_mount-v11.stl" scale="0.001 0.001 0.001" />
             </geometry>
         </collision>
@@ -199,13 +199,13 @@
         </inertial>
         <visual name="ST3215_Servo_Motor-v1_visual">
-            <origin xyz="0.010250000000000035 0.006521312293742278 0.02579524618281096" rpy="1.5707963267948968 0.523598775598299 1.5707963267948972" />
-            <geometry>
-                <mesh filename="${mesh_dir}/ST3215_Servo_Motor-v1.stl" scale="0.001 0.001 0.001" />
+            <origin xyz="0 0 0" rpy="0 0 0" />
+            <geometry>
+                <mesh filename="${mesh_dir}/reauthored/ST3215_Servo_Motor-v1.stl" scale="0.001 0.001 0.001" />
             </geometry>
         </visual>
         <collision name="ST3215_Servo_Motor-v1_collision">
-            <origin xyz="0.010250000000000035 0.006521312293742278 0.02579524618281096" rpy="1.5707963267948968 0.523598775598299 1.5707963267948972" />
-            <geometry>
-                <mesh filename="${mesh_dir}/ST3215_Servo_Motor-v1.stl" scale="0.001 0.001 0.001" />
+            <origin xyz="0 0 0" rpy="0 0 0" />
+            <geometry>
+                <mesh filename="${mesh_dir}/reauthored/ST3215_Servo_Motor-v1.stl" scale="0.001 0.001 0.001" />
             </geometry>
         </collision>
@@ -218,13 +218,13 @@
         </inertial>
         <visual name="omni_wheel_mount-v5_visual">
-            <origin xyz="-0.004838917002787113 -4.662936703425657e-17 0.002793754497239087" rpy="-1.0471975511965974 5.537547822683577e-16 1.5707963267948968" />
-            <geometry>
-                <mesh filename="${mesh_dir}/omni_wheel_mount-v5.stl" scale="0.001 0.001 0.001" />
+            <origin xyz="0 0 0" rpy="0 0 0" />
+            <geometry>
+                <mesh filename="${mesh_dir}/reauthored/omni_wheel_mount-v5.stl" scale="0.001 0.001 0.001" />
             </geometry>
         </visual>
         <collision name="omni_wheel_mount-v5_collision">
-            <origin xyz="-0.004838917002787113 -4.662936703425657e-17 0.002793754497239087" rpy="-1.0471975511965974 5.537547822683577e-16 1.5707963267948968" />
-            <geometry>
-                <mesh filename="${mesh_dir}/omni_wheel_mount-v5.stl" scale="0.001 0.001 0.001" />
+            <origin xyz="0 0 0" rpy="0 0 0" />
+            <geometry>
+                <mesh filename="${mesh_dir}/reauthored/omni_wheel_mount-v5.stl" scale="0.001 0.001 0.001" />
             </geometry>
         </collision>
@@ -237,13 +237,13 @@
         </inertial>
         <visual name="4-Omni-Directional-Wheel_Single_Body-v1_visual">
-            <origin xyz="-0.013748155616372878 -0.007937504497239081 -5.773159728050814e-17" rpy="1.5707963267948974 -1.3089969389957468 2.094395102393195" />
-            <geometry>
-                <mesh filename="${mesh_dir}/4-Omni-Directional-Wheel_Single_Body-v1.stl" scale="0.001 0.001 0.001" />
+            <origin xyz="0 0 0" rpy="0 0 0" />
+            <geometry>
+                <mesh filename="${mesh_dir}/reauthored/4-Omni-Directional-Wheel_Single_Body-v1.stl" scale="0.001 0.001 0.001" />
             </geometry>
         </visual>
         <collision name="4-Omni-Directional-Wheel_Single_Body-v1_collision">
-            <origin xyz="-0.013748155616372878 -0.007937504497239081 -5.773159728050814e-17" rpy="1.5707963267948974 -1.3089969389957468 2.094395102393195" />
-            <geometry>
-                <mesh filename="${mesh_dir}/4-Omni-Directional-Wheel_Single_Body-v1.stl" scale="0.001 0.001 0.001" />
+            <origin xyz="0 0 0" rpy="0 0 0" />
+            <geometry>
+                <mesh filename="${mesh_dir}/reauthored/4-Omni-Directional-Wheel_Single_Body-v1.stl" scale="0.001 0.001 0.001" />
             </geometry>
         </collision>
@@ -256,13 +256,13 @@
         </inertial>
         <visual name="servo_controller_mount-v3_visual">
-            <origin xyz="0.0 0.0 0.006000000000000001" rpy="0.0 -0.0 1.5707963267948966" />
-            <geometry>
-                <mesh filename="${mesh_dir}/servo_controller_mount-v3.stl" scale="0.001 0.001 0.001" />
+            <origin xyz="0 0 0" rpy="0 0 0" />
+            <geometry>
+                <mesh filename="${mesh_dir}/reauthored/servo_controller_mount-v3.stl" scale="0.001 0.001 0.001" />
             </geometry>
         </visual>
         <collision name="servo_controller_mount-v3_collision">
-            <origin xyz="0.0 0.0 0.006000000000000001" rpy="0.0 -0.0 1.5707963267948966" />
-            <geometry>
-                <mesh filename="${mesh_dir}/servo_controller_mount-v3.stl" scale="0.001 0.001 0.001" />
+            <origin xyz="0 0 0" rpy="0 0 0" />
+            <geometry>
+                <mesh filename="${mesh_dir}/reauthored/servo_controller_mount-v3.stl" scale="0.001 0.001 0.001" />
             </geometry>
         </collision>
@@ -275,13 +275,13 @@
         </inertial>
         <visual name="lipo_battery_mount-v3_visual">
-            <origin xyz="-0.01 0.0 -0.0034999999999999966" rpy="3.141592653589793 -0.0 -1.5707963267948968" />
-            <geometry>
-                <mesh filename="${mesh_dir}/lipo_battery_mount-v3.stl" scale="0.001 0.001 0.001" />
+            <origin xyz="0 0 0" rpy="0 0 0" />
+            <geometry>
+                <mesh filename="${mesh_dir}/reauthored/lipo_battery_mount-v3.stl" scale="0.001 0.001 0.001" />
             </geometry>
         </visual>
         <collision name="lipo_battery_mount-v3_collision">
-            <origin xyz="-0.01 0.0 -0.0034999999999999966" rpy="3.141592653589793 -0.0 -1.5707963267948968" />
-            <geometry>
-                <mesh filename="${mesh_dir}/lipo_battery_mount-v3.stl" scale="0.001 0.001 0.001" />
+            <origin xyz="0 0 0" rpy="0 0 0" />
+            <geometry>
+                <mesh filename="${mesh_dir}/reauthored/lipo_battery_mount-v3.stl" scale="0.001 0.001 0.001" />
             </geometry>
         </collision>
@@ -294,13 +294,13 @@
         </inertial>
         <visual name="Battery---Battery-5.2-Ah-DC5521-Plug-v2_visual">
-            <origin xyz="-0.03499999999999998 -4.440892098500626e-18 -1.4432899320127036e-17" rpy="1.224646799147353e-16 -1.5707963267948966 0" />
-            <geometry>
-                <mesh filename="${mesh_dir}/Battery---Battery-5.2-Ah-DC5521-Plug-v2.stl" scale="0.001 0.001 0.001" />
+            <origin xyz="0 0 0" rpy="0 0 0" />
+            <geometry>
+                <mesh filename="${mesh_dir}/reauthored/Battery---Battery-5.2-Ah-DC5521-Plug-v2.stl" scale="0.001 0.001 0.001" />
             </geometry>
         </visual>
         <collision name="Battery---Battery-5.2-Ah-DC5521-Plug-v2_collision">
-            <origin xyz="-0.03499999999999998 -4.440892098500626e-18 -1.4432899320127036e-17" rpy="1.224646799147353e-16 -1.5707963267948966 0" />
-            <geometry>
-                <mesh filename="${mesh_dir}/Battery---Battery-5.2-Ah-DC5521-Plug-v2.stl" scale="0.001 0.001 0.001" />
+            <origin xyz="0 0 0" rpy="0 0 0" />
+            <geometry>
+                <mesh filename="${mesh_dir}/reauthored/Battery---Battery-5.2-Ah-DC5521-Plug-v2.stl" scale="0.001 0.001 0.001" />
             </geometry>
         </collision>
@@ -313,13 +313,13 @@
         </inertial>
         <visual name="94868A713_NO-THREADS_Female-Threaded-Hex-Standoff_visual">
-            <origin xyz="0.0 -1.3010426069826053e-18 -0.025" rpy="3.141592653589793 -0.0 0.0" />
-            <geometry>
-                <mesh filename="${mesh_dir}/94868A713_NO-THREADS_Female-Threaded-Hex-Standoff.stl" scale="0.001 0.001 0.001" />
+            <origin xyz="0 0 0" rpy="0 0 0" />
+            <geometry>
+                <mesh filename="${mesh_dir}/reauthored/94868A713_NO-THREADS_Female-Threaded-Hex-Standoff.stl" scale="0.001 0.001 0.001" />
             </geometry>
         </visual>
         <collision name="94868A713_NO-THREADS_Female-Threaded-Hex-Standoff_collision">
-            <origin xyz="0.0 -1.3010426069826053e-18 -0.025" rpy="3.141592653589793 -0.0 0.0" />
-            <geometry>
-                <mesh filename="${mesh_dir}/94868A713_NO-THREADS_Female-Threaded-Hex-Standoff.stl" scale="0.001 0.001 0.001" />
+            <origin xyz="0 0 0" rpy="0 0 0" />
+            <geometry>
+                <mesh filename="${mesh_dir}/reauthored/94868A713_NO-THREADS_Female-Threaded-Hex-Standoff.stl" scale="0.001 0.001 0.001" />
             </geometry>
         </collision>
@@ -351,13 +351,13 @@
         </inertial>
         <visual name="Bottom-V2-v3_visual">
-            <origin xyz="0.019999999970197697 0.03599999999999999 1.3322676295501878e-16" rpy="4.2524008931839986e-17 3.472469791440238e-17 -3.141592653589793" />
-            <geometry>
-                <mesh filename="${mesh_dir}/Bottom-V2-v3.stl" scale="0.001 0.001 0.001" />
+            <origin xyz="0 0 0" rpy="0 0 0" />
+            <geometry>
+                <mesh filename="${mesh_dir}/reauthored/Bottom-V2-v3.stl" scale="0.001 0.001 0.001" />
             </geometry>
         </visual>
         <collision name="Bottom-V2-v3_collision">
-            <origin xyz="0.019999999970197697 0.03599999999999999 1.3322676295501878e-16" rpy="4.2524008931839986e-17 3.472469791440238e-17 -3.141592653589793" />
-            <geometry>
-                <mesh filename="${mesh_dir}/Bottom-V2-v3.stl" scale="0.001 0.001 0.001" />
+            <origin xyz="0 0 0" rpy="0 0 0" />
+            <geometry>
+                <mesh filename="${mesh_dir}/reauthored/Bottom-V2-v3.stl" scale="0.001 0.001 0.001" />
             </geometry>
         </collision>
@@ -370,13 +370,13 @@
         </inertial>
         <visual name="Top-V2-v2_visual">
-            <origin xyz="0.0003002260252632436 -0.00012500000000001065 0.026499570509487737" rpy="-3.141592653589793 3.851859888774472e-34 -3.141592653589793" />
-            <geometry>
-                <mesh filename="${mesh_dir}/Top-V2-v2.stl" scale="0.001 0.001 0.001" />
+            <origin xyz="0 0 0" rpy="0 0 0" />
+            <geometry>
+                <mesh filename="${mesh_dir}/reauthored/Top-V2-v2.stl" scale="0.001 0.001 0.001" />
             </geometry>
         </visual>
         <collision name="Top-V2-v2_collision">
-            <origin xyz="0.0003002260252632436 -0.00012500000000001065 0.026499570509487737" rpy="-3.141592653589793 3.851859888774472e-34 -3.141592653589793" />
-            <geometry>
-                <mesh filename="${mesh_dir}/Top-V2-v2.stl" scale="0.001 0.001 0.001" />
+            <origin xyz="0 0 0" rpy="0 0 0" />
+            <geometry>
+                <mesh filename="${mesh_dir}/reauthored/Top-V2-v2.stl" scale="0.001 0.001 0.001" />
             </geometry>
         </collision>
@@ -389,13 +389,13 @@
         </inertial>
         <visual name="Camera-Mount-v8_visual">
-            <origin xyz="-0.020000000000000046 0.0 0.0" rpy="0.0 -0.0 1.5707963267948966" />
-            <geometry>
-                <mesh filename="${mesh_dir}/Camera-Mount-v8.stl" scale="0.001 0.001 0.001" />
+            <origin xyz="0 0 0" rpy="0 0 0" />
+            <geometry>
+                <mesh filename="${mesh_dir}/reauthored/Camera-Mount-v8.stl" scale="0.001 0.001 0.001" />
             </geometry>
         </visual>
         <collision name="Camera-Mount-v8_collision">
-            <origin xyz="-0.020000000000000046 0.0 0.0" rpy="0.0 -0.0 1.5707963267948966" />
-            <geometry>
-                <mesh filename="${mesh_dir}/Camera-Mount-v8.stl" scale="0.001 0.001 0.001" />
+            <origin xyz="0 0 0" rpy="0 0 0" />
+            <geometry>
+                <mesh filename="${mesh_dir}/reauthored/Camera-Mount-v8.stl" scale="0.001 0.001 0.001" />
             </geometry>
         </collision>
@@ -408,13 +408,13 @@
         </inertial>
         <visual name="Camera-Model-v3_visual">
-            <origin xyz="-0.01600892660245488 0.0024310699968045314 -0.011393166874206155" rpy="1.7453292519943302 1.3962634015954638 -3.141592653589793" />
-            <geometry>
-                <mesh filename="${mesh_dir}/Camera-Model-v3.stl" scale="0.001 0.001 0.001" />
+            <origin xyz="0 0 0" rpy="0 0 0" />
+            <geometry>
+                <mesh filename="${mesh_dir}/reauthored/Camera-Model-v3.stl" scale="0.001 0.001 0.001" />
             </geometry>
         </visual>
         <collision name="Camera-Model-v3_collision">
-            <origin xyz="-0.01600892660245488 0.0024310699968045314 -0.011393166874206155" rpy="1.7453292519943302 1.3962634015954638 -3.141592653589793" />
-            <geometry>
-                <mesh filename="${mesh_dir}/Camera-Model-v3.stl" scale="0.001 0.001 0.001" />
+            <origin xyz="0 0 0" rpy="0 0 0" />
+            <geometry>
+                <mesh filename="${mesh_dir}/reauthored/Camera-Model-v3.stl" scale="0.001 0.001 0.001" />
             </geometry>
         </collision>
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