Commit message: cad: install v2 wheel cages and reserve 4 mm RobotSkin clearance

File: URDF/LeKiwi.urdf.xacro (robot description, xacro)
@@ -520,10 +520,10 @@
     </link>
     <joint name="base_plate_layer1-v5_baseplate2bottom_mount" type="fixed">
-        <origin xyz="-0.02 -0.1 0.0" rpy="3.141592653589793 -0.0 0.0" />
+        <origin xyz="0.02375 -0.06895 0" rpy="1.57079632679 0 -1.57079632679" />
         <parent link="base_plate_layer1-v5" />
         <child link="drive_motor_mount-v11-2" />
     </joint>
     <joint name="drive_motor_mount-v11-2_Rigid-2" type="fixed">
-        <origin xyz="-0.01214 -0.015999999999999997 -0.0076100000000000004" rpy="3.141592653589793 1.5707963267948966 0" />
+        <origin xyz="0.00555000019073 0.0429865544308 0.0339999998126" rpy="-1.57079632679 1.57079632679 0" />
         <parent link="drive_motor_mount-v11-2" />
         <child link="ST3215_Servo_Motor-v1-2" />
@@ -541,10 +541,10 @@
     </joint>
     <joint name="base_plate_layer1-v5_baseplate2right_mount" type="fixed">
-        <origin xyz="0.07928203 0.022679490000000004 0.0" rpy="0.0 -0.0 0.0" />
+        <origin xyz="0.0478374515909 0.0550431033399 0" rpy="1.57079632679 0 0.523598775598" />
         <parent link="base_plate_layer1-v5" />
         <child link="drive_motor_mount-v11-1" />
     </joint>
     <joint name="drive_motor_mount-v11-1_Rigid-35" type="fixed">
-        <origin xyz="-0.007786400000000002 -0.018513550000000004 0.0076100000000000004" rpy="-7.401486830834375e-17 -1.5707963267948966 0" />
+        <origin xyz="0.00555000203031 0.0429865595601 0.0339999998126" rpy="-3.66519142919 1.57079632679 0" />
         <parent link="drive_motor_mount-v11-1" />
         <child link="ST3215_Servo_Motor-v1-1" />
@@ -562,10 +562,10 @@
     </joint>
     <joint name="base_plate_layer1-v5_baseplate2left_mount" type="fixed">
-        <origin xyz="-0.05928203 0.057320510000000005 0.0" rpy="3.141592653589793 -0.0 0.0" />
+        <origin xyz="-0.0715874515909 0.0139068966601 0" rpy="1.57079632679 2.77555756156e-17 2.61799387799" />
         <parent link="base_plate_layer1-v5" />
         <child link="drive_motor_mount-v11" />
     </joint>
     <joint name="drive_motor_mount-v11_Rigid-39" type="fixed">
-        <origin xyz="0.019926399999999997 -0.0025135499999999933 -0.0076100000000000004" rpy="3.141592653589793 1.5707963267948966 0" />
+        <origin xyz="0.00555000555268 0.0429865554023 0.0339999998126" rpy="-5.75958653158 1.57079632679 0" />
         <parent link="drive_motor_mount-v11" />
         <child link="ST3215_Servo_Motor-v1" />
