Commit message: feat(cad): mount the RobotSkin RPi 5 stack on the upper plate
A 12x10 through plate bolts to real upper-plate holes at the rear right
(pose in sensor_mount_spec.json); the USB carrier and protection table lock
into its ports. The FreeCAD assembly, reauthored meshes and Xacro are
regenerated and the mount checks verify the hole alignment.

Co-Authored-By: Claude Opus 5.5 (1M context) <noreply@anthropic.com>

File: URDF/LeKiwi.urdf.xacro (robot description, xacro)
@@ -516,4 +516,46 @@
             <geometry>
                 <mesh filename="${mesh_dir}/reauthored/astra_pro_compact_mount.stl" scale="0.001 0.001 0.001" />
+            </geometry>
+        </collision>
+    </link>
+    <link name="rpi5_through_plate">
+        <visual name="rpi5_through_plate_visual">
+            <origin xyz="0 0 0" rpy="0 0 0" />
+            <geometry>
+                <mesh filename="${mesh_dir}/reauthored/rpi5_through_plate.stl" scale="0.001 0.001 0.001" />
+            </geometry>
+        </visual>
+        <collision name="rpi5_through_plate_collision">
+            <origin xyz="0 0 0" rpy="0 0 0" />
+            <geometry>
+                <mesh filename="${mesh_dir}/reauthored/rpi5_through_plate.stl" scale="0.001 0.001 0.001" />
+            </geometry>
+        </collision>
+    </link>
+    <link name="rpi5_usb_carrier">
+        <visual name="rpi5_usb_carrier_visual">
+            <origin xyz="0 0 0" rpy="0 0 0" />
+            <geometry>
+                <mesh filename="${mesh_dir}/reauthored/rpi5_usb_carrier.stl" scale="0.001 0.001 0.001" />
+            </geometry>
+        </visual>
+        <collision name="rpi5_usb_carrier_collision">
+            <origin xyz="0 0 0" rpy="0 0 0" />
+            <geometry>
+                <mesh filename="${mesh_dir}/reauthored/rpi5_usb_carrier.stl" scale="0.001 0.001 0.001" />
+            </geometry>
+        </collision>
+    </link>
+    <link name="rpi5_table">
+        <visual name="rpi5_table_visual">
+            <origin xyz="0 0 0" rpy="0 0 0" />
+            <geometry>
+                <mesh filename="${mesh_dir}/reauthored/rpi5_table.stl" scale="0.001 0.001 0.001" />
+            </geometry>
+        </visual>
+        <collision name="rpi5_table_collision">
+            <origin xyz="0 0 0" rpy="0 0 0" />
+            <geometry>
+                <mesh filename="${mesh_dir}/reauthored/rpi5_table.stl" scale="0.001 0.001 0.001" />
             </geometry>
         </collision>
@@ -656,4 +698,19 @@
         <parent link="base_plate_layer2-v3" />
         <child link="astra_pro_compact_mount" />
+    </joint>
+    <joint name="rpi5_through_plate_joint" type="fixed">
+        <origin xyz="0.125 -0.075 0.007" rpy="0.0 0.0 -1.5707963267948966" />
+        <parent link="base_plate_layer2-v3" />
+        <child link="rpi5_through_plate" />
+    </joint>
+    <joint name="rpi5_usb_carrier_joint" type="fixed">
+        <origin xyz="0.0 0.0 0.004" rpy="0 0 0" />
+        <parent link="rpi5_through_plate" />
+        <child link="rpi5_usb_carrier" />
+    </joint>
+    <joint name="rpi5_table_joint" type="fixed">
+        <origin xyz="0.0 0.0 0.004" rpy="0 0 0" />
+        <parent link="rpi5_through_plate" />
+        <child link="rpi5_table" />
     </joint>
     <material name="3d_printed">
